File: kicad-control-board/kicad-control-board.kicad_pcb (KiCad board)
At the start: 2 copper layers, 150 x 180 mm, 62 parts

Commit message: Rework the board for two hemispheres plus a mux, and make it etchable
Board
- Three Teensy 4.1 sockets from a project-local footprint. Rows are 15.24 mm
  apart; the old 17.78 mm was the board width, not the row pitch, so no socket
  could ever line up with a real Teensy.
- Right hemisphere: 9 dual-layer sensors. Left: 7 dual-layer plus 5
  velostat-only loop sensors behind a CD74HC4067 -- the split that fits the 18
  analog inputs a Teensy 4.1 actually has.
- All 21 sensor connectors gathered into two columns on the right edge, with the
  aisle that lets a cable reach the inner column.
- 100 wire landing pads and 74 drum-cable solder pads, so no jumper is soldered
  onto a pin or a component lead that already carries a joint.

Fixed from the previous layout
- Collinear socket rows, which put 11 pairs of different nets on the same hole
- TFT header placed off the board, and buttons overlapping by 3.5 mm
- Bus bars clipping all four mounting holes
- Piezo clamp diodes reversed: cathode was on the ADC node, which forward-biases
  for anything below ~2.6 V and clamps sensing instead of protecting it

Copper sizes for home etching
- Plated pads 2.2 mm, signal tracks 0.8 mm, buses 1.0 mm
- 168 x 240 mm, single-sided: only F.Cu is fabricated, and B.Cu is free to use
  as the wire-jumper guide

Tooling
- jaiba_board_layout.py is the single source of truth for geometry. The pcbnew
  generator and a KiCad-free emitter both consume it.
- make_library / make_teensy_footprint / make_module_footprint generate every
  footprint, so the project needs no KiCad system libraries or install path.
- verify_board.py runs the geometry checks with no KiCad installed.
- route_jumpers.py pre-routes the wire jumpers onto B.Cu as a guide.
- preview_board.py renders the board to SVG to eyeball a floorplan change.

The README documents what is still open, chiefly that the firmware does not yet
match this board: it runs 6 velostat + 6 piezo on a single sensor Teensy, and
the UI only reads Serial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
Parts:
- removed D_PIEZO_TEENSYB0, D_PIEZO_TEENSYB1, D_PIEZO_TEENSYB2, D_PIEZO_TEENSYB3, D_PIEZO_TEENSYB4, D_PIEZO_TEENSYB5, D_PIEZO_TEENSYB6: 1N4148, D_DO-35_SOD27_P7.62mm_Horizontal
- removed J_PIEZO_TEENSYB0, J_PIEZO_TEENSYB1, J_PIEZO_TEENSYB2, J_PIEZO_TEENSYB3, J_PIEZO_TEENSYB4, J_PIEZO_TEENSYB5, J_PIEZO_TEENSYB6, J_VELO_TEENSYA0, J_VELO_TEENSYA1, J_VELO_TEENSYA2, J_VELO_TEENSYA3, J_VELO_TEENSYA4, J_VELO_TEENSYA5, J_VELO_TEENSYA6, J_VELO_TEENSYA7, J_VELO_TEENSYA8: PinHeader_1x02_P2.54mm_Vertical, PinHeader_1x02_P2.54mm_Vertical
- removed J_TEENSYA_R1, J_TEENSYA_R2, J_TEENSYB_R1, J_TEENSYB_R2, J_TEENSYUI_R1, J_TEENSYUI_R2: PinSocket_1x24_P2.54mm_Vertical, PinSocket_1x24_P2.54mm_Vertical
- removed R1_PIEZO_TEENSYB0, R1_PIEZO_TEENSYB1, R1_PIEZO_TEENSYB2, R1_PIEZO_TEENSYB3, R1_PIEZO_TEENSYB4, R1_PIEZO_TEENSYB5, R1_PIEZO_TEENSYB6, R2_PIEZO_TEENSYB0, R2_PIEZO_TEENSYB1, R2_PIEZO_TEENSYB2, R2_PIEZO_TEENSYB3, R2_PIEZO_TEENSYB4, R2_PIEZO_TEENSYB5, R2_PIEZO_TEENSYB6: 10k, R_Axial_DIN0207_L6.3mm_D2.5mm_P10.16mm_Horizontal
- removed R_VELO_TEENSYA0, R_VELO_TEENSYA1, R_VELO_TEENSYA2, R_VELO_TEENSYA3, R_VELO_TEENSYA4, R_VELO_TEENSYA5, R_VELO_TEENSYA6, R_VELO_TEENSYA7, R_VELO_TEENSYA8: 100, R_Axial_DIN0207_L6.3mm_D2.5mm_P10.16mm_Horizontal
- removed SW_CAL_A, SW_CAL_B, SW_CURVE_A, SW_CURVE_B: SW_PUSH_6mm, SW_PUSH_6mm
- added D_L0: 1N4148, D_DO-35_SOD27_P7.62mm_Horizontal, F.Cu at (145.5, 54.0)
- added D_L1: 1N4148, D_DO-35_SOD27_P7.62mm_Horizontal, F.Cu at (145.5, 79.0)
- added D_L2: 1N4148, D_DO-35_SOD27_P7.62mm_Horizontal, F.Cu at (145.5, 104.0)
- added D_L3: 1N4148, D_DO-35_SOD27_P7.62mm_Horizontal, F.Cu at (145.5, 129.0)
- added D_L4: 1N4148, D_DO-35_SOD27_P7.62mm_Horizontal, F.Cu at (145.5, 154.0)
- added D_L5: 1N4148, D_DO-35_SOD27_P7.62mm_Horizontal, F.Cu at (145.5, 179.0)
- added D_L6: 1N4148, D_DO-35_SOD27_P7.62mm_Horizontal, F.Cu at (145.5, 204.0)
- added D_R0: 1N4148, D_DO-35_SOD27_P7.62mm_Horizontal, F.Cu at (113.5, 29.0)
- added D_R1: 1N4148, D_DO-35_SOD27_P7.62mm_Horizontal, F.Cu at (113.5, 54.0)
- added D_R2: 1N4148, D_DO-35_SOD27_P7.62mm_Horizontal, F.Cu at (113.5, 79.0)
- added D_R3: 1N4148, D_DO-35_SOD27_P7.62mm_Horizontal, F.Cu at (113.5, 104.0)
- added D_R4: 1N4148, D_DO-35_SOD27_P7.62mm_Horizontal, F.Cu at (113.5, 129.0)
- added D_R5: 1N4148, D_DO-35_SOD27_P7.62mm_Horizontal, F.Cu at (113.5, 154.0)
- added D_R6: 1N4148, D_DO-35_SOD27_P7.62mm_Horizontal, F.Cu at (113.5, 179.0)
- added D_R7: 1N4148, D_DO-35_SOD27_P7.62mm_Horizontal, F.Cu at (113.5, 204.0)
- added D_R8: 1N4148, D_DO-35_SOD27_P7.62mm_Horizontal, F.Cu at (145.5, 29.0)
- added J_L0: Conn_01x04, PinHeader_1x04_P2.54mm_Vertical, F.Cu at (152.0, 35.0)
- added J_L1: Conn_01x04, PinHeader_1x04_P2.54mm_Vertical, F.Cu at (152.0, 60.0)
- added J_L2: Conn_01x04, PinHeader_1x04_P2.54mm_Vertical, F.Cu at (152.0, 85.0)
- added J_L3: Conn_01x04, PinHeader_1x04_P2.54mm_Vertical, F.Cu at (152.0, 110.0)
- added J_L4: Conn_01x04, PinHeader_1x04_P2.54mm_Vertical, F.Cu at (152.0, 135.0)
- added J_L5: Conn_01x04, PinHeader_1x04_P2.54mm_Vertical, F.Cu at (152.0, 160.0)
- added J_L6: Conn_01x04, PinHeader_1x04_P2.54mm_Vertical, F.Cu at (152.0, 185.0)
- added J_LOOP0: Conn_01x02, PinHeader_1x02_P2.54mm_Vertical, F.Cu at (120.0, 212.0)
- added J_LOOP1: Conn_01x02, PinHeader_1x02_P2.54mm_Vertical, F.Cu at (120.0, 220.0)
- added J_LOOP2: Conn_01x02, PinHeader_1x02_P2.54mm_Vertical, F.Cu at (120.0, 228.0)
- added J_LOOP3: Conn_01x02, PinHeader_1x02_P2.54mm_Vertical, F.Cu at (152.0, 212.0)
- added J_LOOP4: Conn_01x02, PinHeader_1x02_P2.54mm_Vertical, F.Cu at (152.0, 220.0)
- added J_R0: Conn_01x04, PinHeader_1x04_P2.54mm_Vertical, F.Cu at (120.0, 10.0)
- added J_R1: Conn_01x04, PinHeader_1x04_P2.54mm_Vertical, F.Cu at (120.0, 35.0)
- added J_R2: Conn_01x04, PinHeader_1x04_P2.54mm_Vertical, F.Cu at (120.0, 60.0)
- added J_R3: Conn_01x04, PinHeader_1x04_P2.54mm_Vertical, F.Cu at (120.0, 85.0)
- added J_R4: Conn_01x04, PinHeader_1x04_P2.54mm_Vertical, F.Cu at (120.0, 110.0)
- added J_R5: Conn_01x04, PinHeader_1x04_P2.54mm_Vertical, F.Cu at (120.0, 135.0)
- added J_R6: Conn_01x04, PinHeader_1x04_P2.54mm_Vertical, F.Cu at (120.0, 160.0)
- added J_R7: Conn_01x04, PinHeader_1x04_P2.54mm_Vertical, F.Cu at (120.0, 185.0)
- added J_R8: Conn_01x04, PinHeader_1x04_P2.54mm_Vertical, F.Cu at (152.0, 10.0)
- added R1_L0: 10k, R_Axial_DIN0207_L6.3mm_D2.5mm_P10.16mm_Horizontal, F.Cu at (148.0, 45.0)
- added R1_L1: 10k, R_Axial_DIN0207_L6.3mm_D2.5mm_P10.16mm_Horizontal, F.Cu at (148.0, 70.0)
- added R1_L2: 10k, R_Axial_DIN0207_L6.3mm_D2.5mm_P10.16mm_Horizontal, F.Cu at (148.0, 95.0)
- added R1_L3: 10k, R_Axial_DIN0207_L6.3mm_D2.5mm_P10.16mm_Horizontal, F.Cu at (148.0, 120.0)
- added R1_L4: 10k, R_Axial_DIN0207_L6.3mm_D2.5mm_P10.16mm_Horizontal, F.Cu at (148.0, 145.0)
- added R1_L5: 10k, R_Axial_DIN0207_L6.3mm_D2.5mm_P10.16mm_Horizontal, F.Cu at (148.0, 170.0)
- added R1_L6: 10k, R_Axial_DIN0207_L6.3mm_D2.5mm_P10.16mm_Horizontal, F.Cu at (148.0, 195.0)
- added R1_R0: 10k, R_Axial_DIN0207_L6.3mm_D2.5mm_P10.16mm_Horizontal, F.Cu at (116.0, 20.0)
- added R1_R1: 10k, R_Axial_DIN0207_L6.3mm_D2.5mm_P10.16mm_Horizontal, F.Cu at (116.0, 45.0)
- added R1_R2: 10k, R_Axial_DIN0207_L6.3mm_D2.5mm_P10.16mm_Horizontal, F.Cu at (116.0, 70.0)
- added R1_R3: 10k, R_Axial_DIN0207_L6.3mm_D2.5mm_P10.16mm_Horizontal, F.Cu at (116.0, 95.0)
- added R1_R4: 10k, R_Axial_DIN0207_L6.3mm_D2.5mm_P10.16mm_Horizontal, F.Cu at (116.0, 120.0)
- added R1_R5: 10k, R_Axial_DIN0207_L6.3mm_D2.5mm_P10.16mm_Horizontal, F.Cu at (116.0, 145.0)
- added R1_R6: 10k, R_Axial_DIN0207_L6.3mm_D2.5mm_P10.16mm_Horizontal, F.Cu at (116.0, 170.0)
- added R1_R7: 10k, R_Axial_DIN0207_L6.3mm_D2.5mm_P10.16mm_Horizontal, F.Cu at (116.0, 195.0)
- added R1_R8: 10k, R_Axial_DIN0207_L6.3mm_D2.5mm_P10.16mm_Horizontal, F.Cu at (148.0, 20.0)
- added R2_L0: 10k, R_Axial_DIN0207_L6.3mm_D2.5mm_P10.16mm_Horizontal, F.Cu at (137.8, 49.5)
- added R2_L1: 10k, R_Axial_DIN0207_L6.3mm_D2.5mm_P10.16mm_Horizontal, F.Cu at (137.8, 74.5)
- added R2_L2: 10k, R_Axial_DIN0207_L6.3mm_D2.5mm_P10.16mm_Horizontal, F.Cu at (137.8, 99.5)
- added R2_L3: 10k, R_Axial_DIN0207_L6.3mm_D2.5mm_P10.16mm_Horizontal, F.Cu at (137.8, 124.5)
- added R2_L4: 10k, R_Axial_DIN0207_L6.3mm_D2.5mm_P10.16mm_Horizontal, F.Cu at (137.8, 149.5)
- added R2_L5: 10k, R_Axial_DIN0207_L6.3mm_D2.5mm_P10.16mm_Horizontal, F.Cu at (137.8, 174.5)
- added R2_L6: 10k, R_Axial_DIN0207_L6.3mm_D2.5mm_P10.16mm_Horizontal, F.Cu at (137.8, 199.5)
- added R2_R0: 10k, R_Axial_DIN0207_L6.3mm_D2.5mm_P10.16mm_Horizontal, F.Cu at (105.8, 24.5)
- added R2_R1: 10k, R_Axial_DIN0207_L6.3mm_D2.5mm_P10.16mm_Horizontal, F.Cu at (105.8, 49.5)
- added R2_R2: 10k, R_Axial_DIN0207_L6.3mm_D2.5mm_P10.16mm_Horizontal, F.Cu at (105.8, 74.5)
- added R2_R3: 10k, R_Axial_DIN0207_L6.3mm_D2.5mm_P10.16mm_Horizontal, F.Cu at (105.8, 99.5)
- added R2_R4: 10k, R_Axial_DIN0207_L6.3mm_D2.5mm_P10.16mm_Horizontal, F.Cu at (105.8, 124.5)
- added R2_R5: 10k, R_Axial_DIN0207_L6.3mm_D2.5mm_P10.16mm_Horizontal, F.Cu at (105.8, 149.5)
- added R2_R6: 10k, R_Axial_DIN0207_L6.3mm_D2.5mm_P10.16mm_Horizontal, F.Cu at (105.8, 174.5)
- added R2_R7: 10k, R_Axial_DIN0207_L6.3mm_D2.5mm_P10.16mm_Horizontal, F.Cu at (105.8, 199.5)
- added R2_R8: 10k, R_Axial_DIN0207_L6.3mm_D2.5mm_P10.16mm_Horizontal, F.Cu at (137.8, 24.5)
- added RV_L0: 100, R_Axial_DIN0207_L6.3mm_D2.5mm_P10.16mm_Horizontal, F.Cu at (148.0, 37.5)
- added RV_L1: 100, R_Axial_DIN0207_L6.3mm_D2.5mm_P10.16mm_Horizontal, F.Cu at (148.0, 62.5)
- added RV_L2: 100, R_Axial_DIN0207_L6.3mm_D2.5mm_P10.16mm_Horizontal, F.Cu at (148.0, 87.5)
- added RV_L3: 100, R_Axial_DIN0207_L6.3mm_D2.5mm_P10.16mm_Horizontal, F.Cu at (148.0, 112.5)
- added RV_L4: 100, R_Axial_DIN0207_L6.3mm_D2.5mm_P10.16mm_Horizontal, F.Cu at (148.0, 137.5)
- added RV_L5: 100, R_Axial_DIN0207_L6.3mm_D2.5mm_P10.16mm_Horizontal, F.Cu at (148.0, 162.5)
- added RV_L6: 100, R_Axial_DIN0207_L6.3mm_D2.5mm_P10.16mm_Horizontal, F.Cu at (148.0, 187.5)
- added RV_LOOP0: 100, R_Axial_DIN0207_L6.3mm_D2.5mm_P10.16mm_Horizontal, F.Cu at (116.0, 214.5)
- added RV_LOOP1: 100, R_Axial_DIN0207_L6.3mm_D2.5mm_P10.16mm_Horizontal, F.Cu at (116.0, 222.5)
- added RV_LOOP2: 100, R_Axial_DIN0207_L6.3mm_D2.5mm_P10.16mm_Horizontal, F.Cu at (116.0, 230.5)
- added RV_LOOP3: 100, R_Axial_DIN0207_L6.3mm_D2.5mm_P10.16mm_Horizontal, F.Cu at (148.0, 214.5)
- added RV_LOOP4: 100, R_Axial_DIN0207_L6.3mm_D2.5mm_P10.16mm_Horizontal, F.Cu at (148.0, 222.5)
- added RV_R0: 100, R_Axial_DIN0207_L6.3mm_D2.5mm_P10.16mm_Horizontal, F.Cu at (116.0, 12.5)
- added RV_R1: 100, R_Axial_DIN0207_L6.3mm_D2.5mm_P10.16mm_Horizontal, F.Cu at (116.0, 37.5)
- added RV_R2: 100, R_Axial_DIN0207_L6.3mm_D2.5mm_P10.16mm_Horizontal, F.Cu at (116.0, 62.5)
- added RV_R3: 100, R_Axial_DIN0207_L6.3mm_D2.5mm_P10.16mm_Horizontal, F.Cu at (116.0, 87.5)
- added RV_R4: 100, R_Axial_DIN0207_L6.3mm_D2.5mm_P10.16mm_Horizontal, F.Cu at (116.0, 112.5)
- added RV_R5: 100, R_Axial_DIN0207_L6.3mm_D2.5mm_P10.16mm_Horizontal, F.Cu at (116.0, 137.5)
- added RV_R6: 100, R_Axial_DIN0207_L6.3mm_D2.5mm_P10.16mm_Horizontal, F.Cu at (116.0, 162.5)
- added RV_R7: 100, R_Axial_DIN0207_L6.3mm_D2.5mm_P10.16mm_Horizontal, F.Cu at (116.0, 187.5)
- added RV_R8: 100, R_Axial_DIN0207_L6.3mm_D2.5mm_P10.16mm_Horizontal, F.Cu at (148.0, 12.5)
- added SP_L0_1: SolderPad, SolderPad_1x01, F.Cu at (156.5, 35.0)
- added SP_L0_2: SolderPad, SolderPad_1x01, F.Cu at (156.5, 37.5)
- added SP_L0_3: SolderPad, SolderPad_1x01, F.Cu at (156.5, 40.1)
- added SP_L0_4: SolderPad, SolderPad_1x01, F.Cu at (156.5, 42.6)
- added SP_L1_1: SolderPad, SolderPad_1x01, F.Cu at (156.5, 60.0)
- added SP_L1_2: SolderPad, SolderPad_1x01, F.Cu at (156.5, 62.5)
- added SP_L1_3: SolderPad, SolderPad_1x01, F.Cu at (156.5, 65.1)
- added SP_L1_4: SolderPad, SolderPad_1x01, F.Cu at (156.5, 67.6)
- added SP_L2_1: SolderPad, SolderPad_1x01, F.Cu at (156.5, 85.0)
- added SP_L2_2: SolderPad, SolderPad_1x01, F.Cu at (156.5, 87.5)
- added SP_L2_3: SolderPad, SolderPad_1x01, F.Cu at (156.5, 90.1)
- added SP_L2_4: SolderPad, SolderPad_1x01, F.Cu at (156.5, 92.6)
- added SP_L3_1: SolderPad, SolderPad_1x01, F.Cu at (156.5, 110.0)
- added SP_L3_2: SolderPad, SolderPad_1x01, F.Cu at (156.5, 112.5)
- added SP_L3_3: SolderPad, SolderPad_1x01, F.Cu at (156.5, 115.1)
- added SP_L3_4: SolderPad, SolderPad_1x01, F.Cu at (156.5, 117.6)
- added SP_L4_1: SolderPad, SolderPad_1x01, F.Cu at (156.5, 135.0)
- added SP_L4_2: SolderPad, SolderPad_1x01, F.Cu at (156.5, 137.5)
- added SP_L4_3: SolderPad, SolderPad_1x01, F.Cu at (156.5, 140.1)
- added SP_L4_4: SolderPad, SolderPad_1x01, F.Cu at (156.5, 142.6)
- added SP_L5_1: SolderPad, SolderPad_1x01, F.Cu at (156.5, 160.0)
- added SP_L5_2: SolderPad, SolderPad_1x01, F.Cu at (156.5, 162.5)
- added SP_L5_3: SolderPad, SolderPad_1x01, F.Cu at (156.5, 165.1)
- added SP_L5_4: SolderPad, SolderPad_1x01, F.Cu at (156.5, 167.6)
- added SP_L6_1: SolderPad, SolderPad_1x01, F.Cu at (156.5, 185.0)
- added SP_L6_2: SolderPad, SolderPad_1x01, F.Cu at (156.5, 187.5)
- added SP_L6_3: SolderPad, SolderPad_1x01, F.Cu at (156.5, 190.1)
- added SP_L6_4: SolderPad, SolderPad_1x01, F.Cu at (156.5, 192.6)
- added SP_LOOP0_1: SolderPad, SolderPad_1x01, F.Cu at (129.0, 212.0)
- added SP_LOOP0_2: SolderPad, SolderPad_1x01, F.Cu at (129.0, 214.5)
- added SP_LOOP1_1: SolderPad, SolderPad_1x01, F.Cu at (129.0, 220.0)
- added SP_LOOP1_2: SolderPad, SolderPad_1x01, F.Cu at (129.0, 222.5)
- added SP_LOOP2_1: SolderPad, SolderPad_1x01, F.Cu at (129.0, 228.0)
- added SP_LOOP2_2: SolderPad, SolderPad_1x01, F.Cu at (129.0, 230.5)
- added SP_LOOP3_1: SolderPad, SolderPad_1x01, F.Cu at (161.0, 212.0)
- added SP_LOOP3_2: SolderPad, SolderPad_1x01, F.Cu at (161.0, 214.5)
- added SP_LOOP4_1: SolderPad, SolderPad_1x01, F.Cu at (161.0, 220.0)
- added SP_LOOP4_2: SolderPad, SolderPad_1x01, F.Cu at (161.0, 222.5)
- added SP_R0_1: SolderPad, SolderPad_1x01, F.Cu at (124.5, 10.0)
- added SP_R0_2: SolderPad, SolderPad_1x01, F.Cu at (124.5, 12.5)
- added SP_R0_3: SolderPad, SolderPad_1x01, F.Cu at (124.5, 15.1)
- added SP_R0_4: SolderPad, SolderPad_1x01, F.Cu at (124.5, 17.6)
- added SP_R1_1: SolderPad, SolderPad_1x01, F.Cu at (124.5, 35.0)
- added SP_R1_2: SolderPad, SolderPad_1x01, F.Cu at (124.5, 37.5)
- added SP_R1_3: SolderPad, SolderPad_1x01, F.Cu at (124.5, 40.1)
- added SP_R1_4: SolderPad, SolderPad_1x01, F.Cu at (124.5, 42.6)
- added SP_R2_1: SolderPad, SolderPad_1x01, F.Cu at (124.5, 60.0)
- added SP_R2_2: SolderPad, SolderPad_1x01, F.Cu at (124.5, 62.5)
- added SP_R2_3: SolderPad, SolderPad_1x01, F.Cu at (124.5, 65.1)
- added SP_R2_4: SolderPad, SolderPad_1x01, F.Cu at (124.5, 67.6)
- added SP_R3_1: SolderPad, SolderPad_1x01, F.Cu at (124.5, 85.0)
- added SP_R3_2: SolderPad, SolderPad_1x01, F.Cu at (124.5, 87.5)
- added SP_R3_3: SolderPad, SolderPad_1x01, F.Cu at (124.5, 90.1)
- added SP_R3_4: SolderPad, SolderPad_1x01, F.Cu at (124.5, 92.6)
- added SP_R4_1: SolderPad, SolderPad_1x01, F.Cu at (124.5, 110.0)
- added SP_R4_2: SolderPad, SolderPad_1x01, F.Cu at (124.5, 112.5)
- added SP_R4_3: SolderPad, SolderPad_1x01, F.Cu at (124.5, 115.1)
- added SP_R4_4: SolderPad, SolderPad_1x01, F.Cu at (124.5, 117.6)
- added SP_R5_1: SolderPad, SolderPad_1x01, F.Cu at (124.5, 135.0)
- added SP_R5_2: SolderPad, SolderPad_1x01, F.Cu at (124.5, 137.5)
- added SP_R5_3: SolderPad, SolderPad_1x01, F.Cu at (124.5, 140.1)
- added SP_R5_4: SolderPad, SolderPad_1x01, F.Cu at (124.5, 142.6)
- added SP_R6_1: SolderPad, SolderPad_1x01, F.Cu at (124.5, 160.0)
- added SP_R6_2: SolderPad, SolderPad_1x01, F.Cu at (124.5, 162.5)
- added SP_R6_3: SolderPad, SolderPad_1x01, F.Cu at (124.5, 165.1)
- added SP_R6_4: SolderPad, SolderPad_1x01, F.Cu at (124.5, 167.6)
- added SP_R7_1: SolderPad, SolderPad_1x01, F.Cu at (124.5, 185.0)
- added SP_R7_2: SolderPad, SolderPad_1x01, F.Cu at (124.5, 187.5)
- added SP_R7_3: SolderPad, SolderPad_1x01, F.Cu at (124.5, 190.1)
- added SP_R7_4: SolderPad, SolderPad_1x01, F.Cu at (124.5, 192.6)
- added SP_R8_1: SolderPad, SolderPad_1x01, F.Cu at (156.5, 10.0)
- added SP_R8_2: SolderPad, SolderPad_1x01, F.Cu at (156.5, 12.5)
- added SP_R8_3: SolderPad, SolderPad_1x01, F.Cu at (156.5, 15.1)
- added SP_R8_4: SolderPad, SolderPad_1x01, F.Cu at (156.5, 17.6)
- added SW_CAL_L: SW_PUSH, SW_PUSH_6mm, F.Cu at (74.0, 92.0)
- added SW_CAL_R: SW_PUSH, SW_PUSH_6mm, F.Cu at (74.0, 37.0)
- added SW_CURVE_L: SW_PUSH, SW_PUSH_6mm, F.Cu at (74.0, 101.0)
- added SW_CURVE_R: SW_PUSH, SW_PUSH_6mm, F.Cu at (74.0, 46.0)
- added U_L: Teensy4.1, Teensy_4.1, F.Cu at (36.0, 85.0)
- added U_MUX: CD74HC4067, CD74HC4067_Module, F.Cu at (36.0, 130.0)
- added U_R: Teensy4.1, Teensy_4.1, F.Cu at (36.0, 30.0)
- added U_UI: Teensy4.1, Teensy_4.1, F.Cu at (36.0, 165.0)
- added W_L0_PSIG: WirePad, WirePad_1x01, F.Cu at (151.5, 51.5)
- added W_L0_VELO: WirePad, WirePad_1x01, F.Cu at (142.0, 41.5)
- added W_L1_PSIG: WirePad, WirePad_1x01, F.Cu at (151.5, 76.5)
- added W_L1_VELO: WirePad, WirePad_1x01, F.Cu at (142.0, 66.5)
- added W_L2_PSIG: WirePad, WirePad_1x01, F.Cu at (151.5, 101.5)
- added W_L2_VELO: WirePad, WirePad_1x01, F.Cu at (142.0, 91.5)
- added W_L3_PSIG: WirePad, WirePad_1x01, F.Cu at (151.5, 126.5)
- added W_L3_VELO: WirePad, WirePad_1x01, F.Cu at (142.0, 116.5)
- added W_L4_PSIG: WirePad, WirePad_1x01, F.Cu at (151.5, 151.5)
- added W_L4_VELO: WirePad, WirePad_1x01, F.Cu at (142.0, 141.5)
- added W_L5_PSIG: WirePad, WirePad_1x01, F.Cu at (151.5, 176.5)
- added W_L5_VELO: WirePad, WirePad_1x01, F.Cu at (142.0, 166.5)
- added W_L6_PSIG: WirePad, WirePad_1x01, F.Cu at (151.5, 201.5)
- added W_L6_VELO: WirePad, WirePad_1x01, F.Cu at (142.0, 191.5)
- added W_LOOP0_VELO: WirePad, WirePad_1x01, F.Cu at (124.5, 214.5)
- added W_LOOP1_VELO: WirePad, WirePad_1x01, F.Cu at (124.5, 222.5)
- added W_LOOP2_VELO: WirePad, WirePad_1x01, F.Cu at (124.5, 230.5)
- added W_LOOP3_VELO: WirePad, WirePad_1x01, F.Cu at (156.5, 214.5)
- added W_LOOP4_VELO: WirePad, WirePad_1x01, F.Cu at (156.5, 222.5)
- added W_L_0: WirePad, WirePad_1x01, F.Cu at (9.33, 97.1)
- added W_L_1: WirePad, WirePad_1x01, F.Cu at (13.0, 98.3)
- added W_L_14: WirePad, WirePad_1x01, F.Cu at (47.6, 62.5)
- added W_L_15: WirePad, WirePad_1x01, F.Cu at (43.9, 63.7)
- added W_L_16: WirePad, WirePad_1x01, F.Cu at (40.2, 64.8)
- added W_L_17: WirePad, WirePad_1x01, F.Cu at (36.5, 66.0)
- added W_L_18: WirePad, WirePad_1x01, F.Cu at (32.9, 67.1)
- added W_L_19: WirePad, WirePad_1x01, F.Cu at (29.2, 68.3)
- added W_L_20: WirePad, WirePad_1x01, F.Cu at (25.5, 69.4)
- added W_L_21: WirePad, WirePad_1x01, F.Cu at (21.8, 70.6)
- added W_L_22: WirePad, WirePad_1x01, F.Cu at (18.1, 71.7)
- added W_L_23: WirePad, WirePad_1x01, F.Cu at (14.4, 72.9)
- added W_L_24: WirePad, WirePad_1x01, F.Cu at (54.1, 106.3)
- added W_L_3: WirePad, WirePad_1x01, F.Cu at (19.2, 99.4)
- added W_L_38: WirePad, WirePad_1x01, F.Cu at (67.5, 57.9)
- added W_L_39: WirePad, WirePad_1x01, F.Cu at (63.8, 59.1)
- added W_L_4: WirePad, WirePad_1x01, F.Cu at (22.9, 100.6)
- added W_L_40: WirePad, WirePad_1x01, F.Cu at (60.1, 60.2)
- added W_L_41: WirePad, WirePad_1x01, F.Cu at (56.4, 61.4)
- added W_L_5: WirePad, WirePad_1x01, F.Cu at (26.6, 101.7)
- added W_L_6: WirePad, WirePad_1x01, F.Cu at (30.3, 102.9)
- added W_L_7: WirePad, WirePad_1x01, F.Cu at (34.0, 104.0)
- added W_L_8: WirePad, WirePad_1x01, F.Cu at (37.7, 105.2)
- added W_MUX_C0: WirePad, WirePad_1x01, F.Cu at (16.9, 118.0)
- added W_MUX_C1: WirePad, WirePad_1x01, F.Cu at (20.6, 116.9)
- added W_MUX_C2: WirePad, WirePad_1x01, F.Cu at (24.3, 115.8)
- added W_MUX_C3: WirePad, WirePad_1x01, F.Cu at (28.0, 114.6)
- added W_MUX_C4: WirePad, WirePad_1x01, F.Cu at (31.7, 113.5)
- added W_MUX_EN: WirePad, WirePad_1x01, F.Cu at (34.5, 144.2)
- added W_MUX_GND: WirePad, WirePad_1x01, F.Cu at (27.1, 141.9)
- added W_MUX_S0: WirePad, WirePad_1x01, F.Cu at (38.2, 145.4)
- added W_MUX_S1: WirePad, WirePad_1x01, F.Cu at (41.9, 146.6)
- added W_MUX_S2: WirePad, WirePad_1x01, F.Cu at (45.6, 147.7)
- added W_MUX_S3: WirePad, WirePad_1x01, F.Cu at (49.2, 148.8)
- added W_MUX_SIG: WirePad, WirePad_1x01, F.Cu at (52.9, 150.0)
- added W_MUX_VCC: WirePad, WirePad_1x01, F.Cu at (30.8, 143.1)
- added W_R0_PSIG: WirePad, WirePad_1x01, F.Cu at (119.5, 26.5)
- added W_R0_VELO: WirePad, WirePad_1x01, F.Cu at (110.0, 16.5)
- added W_R1_PSIG: WirePad, WirePad_1x01, F.Cu at (119.5, 51.5)
- added W_R1_VELO: WirePad, WirePad_1x01, F.Cu at (110.0, 41.5)
- added W_R2_PSIG: WirePad, WirePad_1x01, F.Cu at (119.5, 76.5)
- added W_R2_VELO: WirePad, WirePad_1x01, F.Cu at (110.0, 66.5)
- added W_R3_PSIG: WirePad, WirePad_1x01, F.Cu at (119.5, 101.5)
- added W_R3_VELO: WirePad, WirePad_1x01, F.Cu at (110.0, 91.5)
- added W_R4_PSIG: WirePad, WirePad_1x01, F.Cu at (119.5, 126.5)
- added W_R4_VELO: WirePad, WirePad_1x01, F.Cu at (110.0, 116.5)
- added W_R5_PSIG: WirePad, WirePad_1x01, F.Cu at (119.5, 151.5)
- added W_R5_VELO: WirePad, WirePad_1x01, F.Cu at (110.0, 141.5)
- added W_R6_PSIG: WirePad, WirePad_1x01, F.Cu at (119.5, 176.5)
- added W_R6_VELO: WirePad, WirePad_1x01, F.Cu at (110.0, 166.5)
- added W_R7_PSIG: WirePad, WirePad_1x01, F.Cu at (119.5, 201.5)
- added W_R7_VELO: WirePad, WirePad_1x01, F.Cu at (110.0, 191.5)
- added W_R8_PSIG: WirePad, WirePad_1x01, F.Cu at (151.5, 26.5)
- added W_R8_VELO: WirePad, WirePad_1x01, F.Cu at (142.0, 16.5)
- added W_R_0: WirePad, WirePad_1x01, F.Cu at (9.33, 42.1)
- added W_R_1: WirePad, WirePad_1x01, F.Cu at (13.0, 43.3)
- added W_R_14: WirePad, WirePad_1x01, F.Cu at (47.6, 7.53)
- added W_R_15: WirePad, WirePad_1x01, F.Cu at (43.9, 8.68)
- added W_R_16: WirePad, WirePad_1x01, F.Cu at (40.2, 9.83)
- added W_R_17: WirePad, WirePad_1x01, F.Cu at (36.5, 11.0)
- added W_R_18: WirePad, WirePad_1x01, F.Cu at (32.9, 12.1)
- added W_R_19: WirePad, WirePad_1x01, F.Cu at (29.2, 13.3)
- added W_R_20: WirePad, WirePad_1x01, F.Cu at (25.5, 14.4)
- added W_R_21: WirePad, WirePad_1x01, F.Cu at (21.8, 15.6)
- added W_R_22: WirePad, WirePad_1x01, F.Cu at (18.1, 16.7)
- added W_R_23: WirePad, WirePad_1x01, F.Cu at (14.4, 17.9)
- added W_R_24: WirePad, WirePad_1x01, F.Cu at (49.5, 46.7)
- added W_R_25: WirePad, WirePad_1x01, F.Cu at (53.2, 47.9)
- added W_R_26: WirePad, WirePad_1x01, F.Cu at (56.9, 49.0)
- added W_R_27: WirePad, WirePad_1x01, F.Cu at (60.6, 50.2)
- added W_R_3: WirePad, WirePad_1x01, F.Cu at (19.2, 44.4)
- added W_R_38: WirePad, WirePad_1x01, F.Cu at (67.5, 2.93)
- added W_R_39: WirePad, WirePad_1x01, F.Cu at (63.8, 4.08)
- added W_R_4: WirePad, WirePad_1x01, F.Cu at (22.9, 45.6)
- added W_R_40: WirePad, WirePad_1x01, F.Cu at (60.1, 5.23)
- added W_R_41: WirePad, WirePad_1x01, F.Cu at (56.4, 6.38)
- added W_UI_0: WirePad, WirePad_1x01, F.Cu at (9.33, 177.1)
- added W_UI_1: WirePad, WirePad_1x01, F.Cu at (13.0, 178.3)
- added W_UI_13: WirePad, WirePad_1x01, F.Cu at (42.1, 150.6)
- added W_UI_14: WirePad, WirePad_1x01, F.Cu at (38.4, 151.7)
- added W_UI_15: WirePad, WirePad_1x01, F.Cu at (34.7, 152.9)
- J_TFT: value PinHeader_1x08_P2.54mm_Vertical -> Conn_01x08
- J_TFT_PWR: value PinHeader_1x02_P2.54mm_Vertical -> Conn_01x02
- MH1, MH2, MH3, MH4: value MountingHole_3.2mm_M3 -> MountingHole
- moved MH4 61.4 mm to (162.0, 234.0)
- moved MH3 59.0 mm to (6.00, 234.0)
- moved MH2 17.0 mm to (162.0, 6.00)
- moved J_TFT 16.6 mm to (22.0, 181.6), turned to 90 degrees
- moved J_TFT_PWR 13.7 mm to (14.0, 181.6), turned to 90 degrees
- moved MH1 1.41 mm to (6.00, 6.00)
Routing:
- net L_PSIG6: track 0.00 -> 276.4 mm
- net R_PSIG6: track 0.00 -> 273.9 mm
- net L_VELO6: track 0.00 -> 262.9 mm
- net LOOP_VELO4: track 0.00 -> 260.7 mm
- net R_VELO6: track 0.00 -> 260.4 mm
- net LOOP_VELO3: track 0.00 -> 254.8 mm
- net L_PSIG5: track 0.00 -> 252.6 mm
- net R_PSIG7: track 0.00 -> 251.9 mm
- net R_PSIG5: track 0.00 -> 249.4 mm
- net LOOP_VELO2: track 0.00 -> 239.9 mm
- net L_VELO5: track 0.00 -> 238.5 mm
- net R_VELO5: track 0.00 -> 236.6 mm
- net R_VELO7: track 0.00 -> 233.8 mm
- net LOOP_VELO1: track 0.00 -> 232.2 mm
- net L_PSIG4: track 0.00 -> 226.9 mm
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Other:
- board size 150 x 180 mm -> 168 x 240 mm

Commit message: Re-fit to 150 x 260 mm, widen the drum pads, add encoder headers
Board outline
- 150 x 260 mm, fixed by the enclosure, so it is a constraint rather than an
  outcome. Reaching 150 wide was a re-flow of the left region, not of the cell
  columns: the old layout had ~30 mm of dead space between the Teensys and the
  buses. Teensy x 36->32, buses 92/100->66/71, columns 104/136->78/114.
- The extra 20 mm of height went into the cell row pitch (25 -> 27 mm) and a
  button cluster at the bottom left. The buttons had to move anyway: their old
  spot was exactly where the buses needed to go, and the gap there is now under
  3 mm, too narrow for a 9.5 mm switch.

Drum-cable solder pads
- 4.0 x 2.0 mm -> 8.0 x 2.0 mm. Per connection that is now 19.8 mm2, 5.2x the
  through-hole pad alone, and an 8 mm run of copper to solder the cable along.
- The extra length pushed the loop cells' jumper pads out of the strip they
  shared with the drum pads, so those moved below (row pitch 8 -> 11 mm) and
  column B moved 114 mm to keep the aisle between the columns.

Encoder expansion headers
- J_ENC_A (10 pins), J_ENC_B (9), J_ENC_C (9): 26 free UI Teensy digital pins,
  including all 16 analog-capable ones. A carries GND and 3V3 taken from the
  Teensy's own ROW1 pins, so no bus has to be tapped.
- Three headers rather than one because each pin row is a wall: a track cannot
  pass between two 2.2 mm pads on a 2.54 mm pitch, so nothing reaches ROW1 from
  below. Each header sits on the side of the row it serves and every trace is a
  straight vertical -- pin for pin, no crossings, no jumpers, no vias.
- J_ENC_A sits 5.5 mm higher than B to fit between the mux's channel extension
  pads below and the UART landing pad for pin 15 above.

Fixes along the way
- make_pin_header builds a vertical header (pads along Y), so the headers ran
  down into the Teensy until they were rotated 90 degrees.
- README had two near-identical "Board geometry" sections; merged.

No multiplexer is needed for knob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
Parts:
- added J_ENC_A: Conn_01x10, PinHeader_1x10_P2.54mm_Vertical, F.Cu at (5.33, 148.5)
- added J_ENC_B: Conn_01x09, PinHeader_1x09_P2.54mm_Vertical, F.Cu at (40.9, 154.0)
- added J_ENC_C: Conn_01x09, PinHeader_1x09_P2.54mm_Vertical, F.Cu at (40.9, 190.0)
- moved SW_CAL_R 180.7 mm to (10.0, 206.0)
- moved SW_CURVE_R 166.5 mm to (28.0, 206.0)
- moved SW_CAL_L 148.5 mm to (10.0, 226.0)
- moved SW_CURVE_L 133.2 mm to (28.0, 226.0)
- moved SP_LOOP2_1 33.7 mm to (100.5, 246.0)
- moved SP_LOOP2_2 33.7 mm to (100.5, 248.5)
- moved SP_LOOP1_1 32.2 mm to (100.5, 235.0)
- moved SP_LOOP1_2 32.2 mm to (100.5, 237.5)
- moved W_LOOP2_VELO 31.7 mm to (100.5, 251.2)
- moved J_LOOP2 31.6 mm to (94.0, 246.0)
- moved RV_LOOP2 31.6 mm to (90.0, 248.5)
- moved SP_LOOP0_1 30.9 mm to (100.5, 224.0)
- moved SP_LOOP0_2 30.9 mm to (100.5, 226.5)
- moved J_LOOP1 30.0 mm to (94.0, 235.0)
- moved RV_LOOP1 30.0 mm to (90.0, 237.5)
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Connections:
- U_UI pad 16: (no net) -> UI16
- U_UI pad 17: (no net) -> UI17
- U_UI pad 18: (no net) -> UI18
- U_UI pad 19: (no net) -> UI19
- U_UI pad 20: (no net) -> UI20
- U_UI pad 21: (no net) -> UI21
- U_UI pad 22: (no net) -> UI22
- U_UI pad 23: (no net) -> UI23
- U_UI pad 24: (no net) -> UI24
- U_UI pad 25: (no net) -> UI25
- U_UI pad 26: (no net) -> UI26
- U_UI pad 27: (no net) -> UI27
- U_UI pad 28: (no net) -> UI28
- U_UI pad 29: (no net) -> UI29
- U_UI pad 30: (no net) -> UI30
- U_UI pad 31: (no net) -> UI31
- U_UI pad 32: (no net) -> UI32
- U_UI pad 33: (no net) -> UI33
- U_UI pad 34: (no net) -> UI34
- U_UI pad 35: (no net) -> UI35
- U_UI pad 36: (no net) -> UI36
- U_UI pad 37: (no net) -> UI37
- U_UI pad 38: (no net) -> UI38
- U_UI pad 39: (no net) -> UI39
- U_UI pad 40: (no net) -> UI40
- U_UI pad 41: (no net) -> UI41
Routing:
- net BTN_CURVE_R: track 62.6 -> 214.4 mm
- net BTN_CAL_R: track 70.0 -> 192.6 mm
- net BTN_CURVE_L: track 63.3 -> 180.1 mm
- net BTN_CAL_L: track 70.0 -> 157.7 mm
- net GND: track 315.7 -> 376.6 mm
- net 3V3: track 354.8 -> 403.1 mm
- net L_PSIG1: track 175.1 -> 149.7 mm
- net L_VELO1: track 167.1 -> 142.4 mm
- net R_PSIG0: track 134.1 -> 111.9 mm
- net R_PSIG1: track 158.5 -> 138.2 mm
- net L_PSIG0: track 179.2 -> 158.9 mm
- net R_VELO0: track 122.0 -> 102.4 mm
- net R_PSIG2: track 182.4 -> 163.3 mm
- net R_PSIG8: track 166.5 -> 148.1 mm
- net L_VELO0: track 184.9 -> 166.6 mm
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Other:
- board size 168 x 240 mm -> 150 x 260 mm

Commit message: Ground in copper and a grounded electrostatic shield
Ground wiring, cut in copper
- Each dual-layer cell had three separate ground points: the connector's GND
  (with its drum pad already stubbed to it), the piezo divider's GND, and the
  velostat pulldown's GND. A short F.Cu run joins all three, going the long way
  round because the pulldown's GND pad sits behind the piezo node with the psig
  feed running down that same column.
- Ground drops from 63 wire connections to 31.

Rejected: a ground pour
- tools/check_pour.py measures whether a pour would actually connect, rather
  than asserting it. It rasterises the board, models thermal spokes (a pad need
  not sit IN the pour -- a spoke crosses its clearance ring, which at 2.54 mm
  pitch with 2.2 mm pads is the only way most pads ever connect), and partitions
  the plane.
- Result: even with spokes, one layer fragments ground into 15 pieces. Every
  signal track is a wall through the plane and ~600 of them partition it. So a
  pour cannot be the ground return path here, and grounding a fragmented one
  would put parallel paths beside the high-impedance piezo nodes.
- 3V3 remains the largest hand-wiring item at 42. The diode's 3V3 pad sits in a
  pocket -- the psig feed crosses the cell above it, the cell ends below it, and
  the drum stubs wall off the right -- so joining it needs a cell re-layout, not
  another trace.

The shield
- The F.Cu copper fill is tied to GND and acts as a coplanar shield/guard around
  the high-impedance piezo nodes. It MUST be grounded: floating copper
  re-radiates and capacitively couples onto the very nodes it sits beside.
- island_removal_mode 2 so no fragment is left floating.
- Fragmentation, which rules the fill out as a return path, is fine for a
  shield: each piece only needs grounding, not joining to the others.
  15 of 146 regions reach ground = 292.81 cm2 of useful shield (75% of the
  board), with 4.52 cm2 floating and removed.
- This is a coplanar guard, not a true planar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
Routing:
- net GND: track 376.6 -> 904.6 mm
- net 3V3: track 403.1 -> 401.1 mm
- added copper zone on F.Cu, net GND
